File: pcb/usbc-hub.brd (EAGLE design)
At the start: 100 x 60 mm, 10 parts, among them U1 USB5826, U2 HD3SS3220, U3 MIC24045

Commit message: Schematic almost complete
Parts:
- added C1, C2, C3, C4, C5, C6, C7, C8: 100nF, Capacitor:CAP0603
- added C10, C11, C12, C13, C14, C9: 100uF, Capacitor:CAP1206
- added C15, C16: (no value), Capacitor:CAP0603
- added D1, D2: DSK24, Generic Diode:SOD-123F
- added Q1, Q2, Q3, Q4: AO3401, Alpha Omega:SOT23
- added R1, R20, R22: 50K Ohms, Resistor:RES0603
- added R10, R8: 47K Ohms, Resistor:RES0603
- added R11, R9: 8.2K Ohms, Resistor:RES0603
- added R12, R13, R6, R7: 22K Ohms, Resistor:RES0603
- added R14, R15, R16, R17, R18, R19, R29, R30, R31, R35, R36, R37, R38, R39, R40, R41, R42, R43, R44, R45, R46: 10K Ohms, Resistor:RES0603
- added R2, R21, R23: 100K Ohms, Resistor:RES0603
- added R24, R26: 35.7K Ohms, Resistor:RES0603
- added R25, R27: 5.1K Ohms, Resistor:RES0603
- added R28: 12K Ohms, Resistor:RES0603
- added R3: 4.7K Ohms, Resistor:RES0603
- added R32, R33, R34, R5: 200K Ohms, Resistor:RES0603
- added R4: 900K Ohms, Resistor:RES0603
- added SJ1: SJCS, Solder Jumper:SJC_S
- added U10: USB5826, Microchip:VQFN100
- added U11: MIC24045, Microchip:FQFN20
- added U4, U5, U8, U9: MIC2019, Microchip:SOT23-6
- added U6, U7: UTC2000, Microchip:QFN16
- added X1: 25 MHz, Crystal:4-SMD-3225
- U1: value USB5826 -> HD3SS3220; device Microchip:VQFN100 -> Texas Instruments:WQFN30
- U2: value HD3SS3220 -> MIC2019; device Texas Instruments:WQFN30 -> Microchip:SOT23-6
- U3: value MIC24045 -> MIC2019; device Microchip:FQFN20 -> Microchip:SOT23-6
- USB2: value USB-C-24P-SMD-FLAT-SIDE -> USB3-A-TH-FLAT-SIDE; device USB Connector:USB-C-24P-SMD-FLAT-SIDE -> USB Connector:USB3-A-TH-FLAT-SIDE
- USB4: value USB3-A-TH-FLAT-SIDE -> USB-A-TH-FLAT-SIDE; device USB Connector:USB3-A-TH-FLAT-SIDE -> USB Connector:USB-A-TH-FLAT-SIDE
- USB6: value USB-A-TH-FLAT-SIDE -> USB-C-24P-SMD-FLAT-SIDE; device USB Connector:USB-A-TH-FLAT-SIDE -> USB Connector:USB-C-24P-SMD-FLAT-SIDE
- moved U3 131.4 mm to (-40.0, -22.5)
- moved U2 98.7 mm to (-40.0, -29.9)
- moved USB2 76.0 mm to (28.3, 15.3)
- moved USB6 61.6 mm to (97.4, 47.0), turned to 180 degrees
- moved USB1 44.9 mm to (2.60, 47.0), turned to 0 degrees
- moved USB7 44.9 mm to (9.30, 2.60), turned to 90 degrees
- moved U1 35.8 mm to (18.8, 47.1), turned to 180 degrees
- moved USB4 20.3 mm to (48.0, 10.2), turned to 90 degrees
Connections:
- removed net VDD12: U1.10, U1.17, U1.26, U1.32, U1.39, U1.47, U1.59, U1.78, U1.83, U1.90, U1.98
- removed net VDD33: U1.2, U1.27, U1.42, U1.5, U1.54, U1.64, U1.72, U1.93
- removed net VSS: U1.101
- new net !DN1_VC1_EN: Q1.1, R14.1, U6.9
- new net !DN1_VC2_EN: Q3.1, R16.1, U6.8
- new net !DN2_VC1_EN: Q2.1, R15.1, U7.9
- new net !DN2_VC2_EN: Q4.1, R17.1, U7.8
- new net !SPI_CS: R34.2, U10.68
- new net 1V2: U10.10, U10.17, U10.26, U10.32, U10.39, U10.47, U10.59, U10.78, U10.83, U10.90, U10.98
- new net 3V3: R18.2, R19.2, R29.2, R30.2, R31.2, R5.2, U1.8, U10.2, U10.27, U10.42, U10.5, U10.54, U10.64, U10.72, U10.93
- new net 5V0: D1.A, D2.A, R10.2, R12.2, R13.2, R14.2, R15.2, R16.2, R17.2, R6.2, R7.2, R8.2, U1.30, U6.16, U7.16, U8.1, U9.1
- new net DN1_ATTACH: R20.1, R21.2, U10.73
- new net DN1_CC1: Q1.3, R6.1, U6.7, USB6.A5
- new net DN1_CC2: Q3.3, R12.1, U6.6, USB6.B5
- new net DN1_D+: R35.2, U10.6, USB6.A6, USB6.B6
- new net DN1_D-: R38.2, U10.7, USB6.A7, USB6.B7
- new net DN1_DIR: R18.1, U10.50, U6.11
- new net DN1_EN/!OC_DET: U10.70, U6.1, U6.3, U8.4
- new net DN1_PWR_EN: R20.2, U6.10, U8.3
- new net DN1_RXA+: U10.11, USB6.B11
- new net DN1_RXA-: U10.12, USB6.B10
- new net DN1_RXB+: U10.18, USB6.A11
- new net DN1_RXB-: U10.19, USB6.A10
- new net DN1_TXA+: U10.8, USB6.A2
- new net DN1_TXA-: U10.9, USB6.A3
- new net DN1_TXB+: U10.15, USB6.B2
- new net DN1_TXB-: U10.16, USB6.B3
- new net DN1_VMON: R24.1, R25.2, U6.12
- new net DN2_ATTACH: R22.1, R23.2, U10.56
- new net DN2_CC1: Q2.3, R7.1, U7.7, USB7.A5
- new net DN2_CC2: Q4.3, R13.1, U7.6, USB7.B5
- new net DN2_D+: R41.2, U10.28, USB7.A6, USB7.B6
- new net DN2_D-: R44.2, U10.29, USB7.A7, USB7.B7
- new net DN2_DIR: R19.1, U10.71, U7.11
- new net DN2_EN/!OC_DET: U10.58, U7.1, U7.3, U9.4
- new net DN2_PWR_EN: R22.2, U7.10, U9.3
- new net DN2_PWR_EN1: R1.2
- new net DN2_RXA+: U10.33, USB7.B11
- new net DN2_RXA-: U10.34, USB7.B10
- new net DN2_RXB+: U10.40, USB7.A11
- new net DN2_RXB-: U10.41, USB7.A10
- new net DN2_TXA+: U10.30, USB7.A2
- new net DN2_TXA-: U10.31, USB7.A3
- new net DN2_TXB+: U10.37, USB7.B2
- new net DN2_TXB-: U10.38, USB7.B3
- new net DN2_VMON: R26.1, R27.2, U7.12
- new net DN3_D+: R36.2, U10.43, USB2.D+
- new net DN3_D-: R39.2, U10.44, USB2.D-
- new net DN3_EN/!OC_DET: U10.52, U2.3, U2.4
- new net DN3_RX+: U10.48, USB2.RX+
- new net DN3_RX-: U10.49, USB2.RX-
- new net DN3_TX+: U10.45, USB2.TX+
- new net DN3_TX-: U10.46, USB2.TX-
- new net DN4_D+: R42.2, U10.86, USB3.D+
- new net DN4_D-: R45.2, U10.87, USB3.D-
- new net DN4_EN/!OC_DET: U10.51, U3.3, U3.4
- new net DN4_RX+: U10.91, USB3.RX+
- new net DN4_RX-: U10.92, USB3.RX-
- new net DN4_TX+: U10.88, USB3.TX+
- new net DN4_TX-: U10.89, USB3.TX-
- new net DN5_D+: R37.2, U10.13, USB4.D+
- new net DN5_D-: R40.2, U10.14, USB4.D-
- new net DN5_EN/!OC_DET: U10.62, U4.3, U4.4
- new net DN6_D+: R43.2, U10.35, USB5.D+
- new net DN6_D-: R46.2, U10.36, USB5.D-
- new net DN6_EN/!OC_DET: U10.57, U5.3, U5.4
- new net GND: C10.2, C11.2, C12.2, C13.2, C14.2, C15.1, C16.2, C9.2, R11.1, R2.1, R21.1, R23.1, R25.1, R27.1, R28.1, R3.1, R32.1, R33.1, R34.1, R35.1, R36.1, R37.1, R38.1, R39.1, R40.1, R41.1, R42.1, R43.1, R44.1, R45.1, R46.1, R9.1, U1.12, U1.13, U1.28, U1.29, U1.31, U10.101, U10.23, U10.61, U10.63, U6.13, U6.17, U7.13, U7.17, USB1.A1, USB1.A12, USB1.B1, USB1.B12, USB1.SHIELD@0, USB1.SHIELD@1, USB1.SHIELD@2, USB1.SHIELD@3, USB2.GND, USB2.P$10, USB2.P$11, USB2.SS_GND, USB3.GND, USB3.P$10, USB3.P$11, USB3.SS_GND, USB4.GND, USB4.P$5, USB4.P$6, USB5.GND, USB5.P$5, USB5.P$6, USB6.A1, USB6.A12, USB6.B1, USB6.B12, USB6.SHIELD@0, USB6.SHIELD@1, USB6.SHIELD@2, USB6.SHIELD@3, USB7.A1, USB7.A12, USB7.B1, USB7.B12, USB7.SHIELD@0, USB7.SHIELD@1, USB7.SHIELD@2, USB7.SHIELD@3, X1.2, X1.4
- new net I2C_SCL: R30.1, U10.75
- new net I2C_SDA: R31.1, U10.74
- new net N$1: C1.2, U1.17
- new net N$10: R3.2, U1.4
- new net N$11: C14.1, U9.6, USB7.A4, USB7.A9, USB7.B4, USB7.B9
- new net N$12: C13.1, R24.2, U8.6, USB6.A4, USB6.A9, USB6.B4, USB6.B9
- new net N$13: C9.1, U2.6, USB2.VBUS
- new net N$14: C12.1, U5.6, USB5.VBUS
- new net N$15: C11.1, U4.6, USB4.VBUS
- new net N$16: C10.1, U3.6, USB3.VBUS
- new net N$17: C16.1, U10.4, X1.3
- new net N$18: C15.2, U10.3, X1.1
- new net N$19: R32.2, U10.20
- new net N$2: C2.2, U1.16
- new net N$20: R29.1, U10.25
- new net N$21: D2.C, Q2.2, Q4.2
- new net N$22: R28.2, U10.1
- new net N$23: D1.C, Q1.2, Q3.2
- new net N$24: R10.1, R11.2, U7.2
- new net N$25: R8.1, R9.2, U6.2
- new net N$26: R26.2
- new net N$27: R5.1, U1.11
- new net N$3: C3.2, U1.21
- new net N$4: C4.2, U1.20
- new net N$5: C5.2, U1.15
- new net N$6: C6.2, U1.14
- new net N$7: C7.2, U1.19
- new net N$8: C8.2, U1.18
- new net N$9: R4.1, U1.5
- new net SPI_MISO: R33.2, U10.67
- new net SPI_MOSI: U10.66
- new net SPI_SCK: U10.65
- new net UP_ATTACH: SJ1.2, U10.76
- new net UP_CC1: U1.2, USB1.A5
- new net UP_CC2: U1.1, USB1.B5
- new net UP_D+: U10.94, USB1.A6, USB1.B6
- new net UP_D-: U10.95, USB1.A7, USB1.B7
- new net UP_RX+: U1.9, U10.99
- new net UP_RX-: U1.10, U10.100
- new net UP_RX1+: C5.1, USB1.B11
- new net UP_RX1-: C6.1, USB1.B10
- new net UP_RX2+: C7.1, USB1.A11
- new net UP_RX2-: C8.1, USB1.A10
- new net UP_TX+: U1.6, U10.96
- new net UP_TX-: U1.7, U10.97
- new net UP_TX1+: C1.1, USB1.A2
- new net UP_TX1-: C2.1, USB1.A3
- new net UP_TX2+: C3.1, USB1.B2
- new net UP_TX2-: C4.1, USB1.B3
- new net UP_VBUS_DET: R1.1, R2.2, SJ1.1, U10.24
- new net VBUS: R4.2, USB1.A4, USB1.A9, USB1.B4, USB1.B9

Commit message: Work on power
Parts:
- added F1, F2: (no value), PTC Fuses:1812
- added J1: DCJACK, DC Jack:DC-050
- added R47, R48: 165 Ohms, Resistor:RES0603
- added U12: MIC23159, Microchip:VQFN20
- U11: value MIC24045 -> MIC24045-KD
- moved D2 352.6 mm to (10.7, 17.6)
- moved Q4 350.3 mm to (9.50, 21.1)
- moved Q2 346.4 mm to (9.50, 24.4)
- moved D1 340.8 mm to (69.3, 46.8), turned to 180 degrees
- moved Q3 335.9 mm to (76.5, 44.7)
- moved Q1 332.2 mm to (76.5, 48.1)
- moved U9 301.5 mm to (5.60, 17.3)
- moved U8 161.1 mm to (84.5, 42.7)
- moved U5 140.9 mm to (84.8, 20.8), turned to 270 degrees
- moved U6 138.0 mm to (84.3, 48.6)
- moved X1 132.5 mm to (37.3, 40.8)
- moved U3 113.4 mm to (64.1, 22.4), turned to 270 degrees
- moved U4 102.3 mm to (43.1, 22.4), turned to 270 degrees
- moved U2 82.1 mm to (23.5, 22.2), turned to 270 degrees
- moved U11 59.7 mm to (18.5, 35.3)
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Connections:
- new net N$28: R47.1, U8.5
- new net N$29: R48.1, U9.5
- net 5V0: now also F1.1
- net GND: now also R47.2, R48.2, U8.2, U9.2
- net VBUS: now also F1.2
Routing:
- added copper zone on layer 1, net GND
- added copper zone on layer 16, net GND
