File: pcb/usbc-hub.sch (EAGLE design)
At the start: 10 parts, among them U1 USB5826, U2 HD3SS3220, U3 MIC24045

Commit message: Schematic almost complete
Parts:
- added C1, C2, C3, C4, C5, C6, C7, C8: 100nF, Capacitor:CAPACITOR-0603
- added C10, C11, C12, C13, C14, C9: 100uF, Capacitor:CAPACITOR-1206
- added C15, C16: (no value), Capacitor:CAPACITOR-0603
- added D1, D2: DSK24, Generic Diode:DSK24
- added Q1, Q2, Q3, Q4: AO3401, Alpha Omega:AO3401
- added R1, R20, R22: 50K Ohms, Resistor:RESISTOR-0603
- added R10, R8: 47K Ohms, Resistor:RESISTOR-0603
- added R11, R9: 8.2K Ohms, Resistor:RESISTOR-0603
- added R12, R13, R6, R7: 22K Ohms, Resistor:RESISTOR-0603
- added R14, R15, R16, R17, R18, R19, R29, R30, R31, R35, R36, R37, R38, R39, R40, R41, R42, R43, R44, R45, R46: 10K Ohms, Resistor:RESISTOR-0603
- added R2, R21, R23: 100K Ohms, Resistor:RESISTOR-0603
- added R24, R26: 35.7K Ohms, Resistor:RESISTOR-0603
- added R25, R27: 5.1K Ohms, Resistor:RESISTOR-0603
- added R28: 12K Ohms, Resistor:RESISTOR-0603
- added R3: 4.7K Ohms, Resistor:RESISTOR-0603
- added R32, R33, R34, R5: 200K Ohms, Resistor:RESISTOR-0603
- added R4: 900K Ohms, Resistor:RESISTOR-0603
- added SJ1: SJCS, Solder Jumper:SJCS
- added U10: USB5826, Microchip:USB5826
- added U11: MIC24045, Microchip:MIC24045
- added U4, U5, U8, U9: MIC2019, Microchip:MIC2019
- added U6, U7: UTC2000, Microchip:UTC2000
- added X1: 25 MHz, Crystal:CRYSTAL_4P
- U1: value USB5826 -> HD3SS3220; device Microchip:USB5826 -> Texas Instruments:HD3SS3220
- U2: value HD3SS3220 -> MIC2019; device Texas Instruments:HD3SS3220 -> Microchip:MIC2019
- U3: value MIC24045 -> MIC2019; device Microchip:MIC24045 -> Microchip:MIC2019
- USB2: value USB-C-24P-SMD-FLAT-SIDE -> USB3-A-TH-FLAT-SIDE; device USB Connector:USB-C-24P-SMD-FLAT-SIDE -> USB Connector:USB3-A-TH-FLAT-SIDE
- USB4: value USB3-A-TH-FLAT-SIDE -> USB-A-TH-FLAT-SIDE; device USB Connector:USB3-A-TH-FLAT-SIDE -> USB Connector:USB-A-TH-FLAT-SIDE
- USB6: value USB-A-TH-FLAT-SIDE -> USB-C-24P-SMD-FLAT-SIDE; device USB Connector:USB-A-TH-FLAT-SIDE -> USB Connector:USB-C-24P-SMD-FLAT-SIDE
Connections:
- new net !DN1_VC1_EN: Q1.G, R14.1, U6.!VCONN1!/!1.5A
- new net !DN1_VC2_EN: Q3.G, R16.1, U6.!VCONN2!/!LEGACY
- new net !DN2_VC1_EN: Q2.G, R15.1, U7.!VCONN1!/!1.5A
- new net !DN2_VC2_EN: Q4.G, R17.1, U7.!VCONN2!/!LEGACY
- new net !SPI_CS: R34.2, U10.GPIO7/!SPI_CE!/CFG_NON_REM
- new net 1V2: U10.VDD12@0, U10.VDD12@1, U10.VDD12@10, U10.VDD12@2, U10.VDD12@3, U10.VDD12@4, U10.VDD12@5, U10.VDD12@6, U10.VDD12@7, U10.VDD12@8, U10.VDD12@9
- new net 3V3: R18.2, R19.2, R29.2, R30.2, R31.2, R5.2, U1.VCC33, U10.VDD33@0, U10.VDD33@1, U10.VDD33@2, U10.VDD33@3, U10.VDD33@4, U10.VDD33@5, U10.VDD33@6, U10.VDD33@7
- new net 5V0: D1.A, D2.A, R10.2, R12.2, R13.2, R14.2, R15.2, R16.2, R17.2, R6.2, R7.2, R8.2, U1.VDD5, U6.VDD, U7.VDD, U8.VIN, U9.VIN
- new net DN1_ATTACH: R20.1, R21.2, U10.GPIO1/C_ATTACH1/ATTACHMUX1A
- new net DN1_CC1: Q1.D, R6.1, U6.CC1, USB6.CC1
- new net DN1_CC2: Q3.D, R12.1, U6.CC2, USB6.CC2
- new net DN1_D+: R35.2, U10.USB2DN1_D+, USB6.D+
- new net DN1_D-: R38.2, U10.USB2DN1_D-, USB6.D-
- new net DN1_DIR: R18.1, U10.GPIO65/AB1/ATTACHMUX1B, U6.!FLIPPED
- new net DN1_EN/!OC_DET: U10.GPIO17/PRT_CTL1, U6.!OCS, U6.EN, U8.!FAULT
- new net DN1_PWR_EN: R20.2, U6.VBUS_EN/!3.0A, U8.EN
- new net DN1_RXA+: U10.USB3DN1_RXA+, USB6.RX1+
- new net DN1_RXA-: U10.USB3DN1_RXA-, USB6.RX1-
- new net DN1_RXB+: U10.USB3DN1_RXB+, USB6.RX2+
- new net DN1_RXB-: U10.USB3DN1_RXB-, USB6.RX2-
- new net DN1_TXA+: U10.USB3DN1_TXA+, USB6.TX1+
- new net DN1_TXA-: U10.USB3DN1_TXA-, USB6.TX1-
- new net DN1_TXB+: U10.USB3DN1_TXB+, USB6.TX2+
- new net DN1_TXB-: U10.USB3DN1_TXB-, USB6.TX2-
- new net DN1_VMON: R24.1, R25.2, U6.VMON
- new net DN2_ATTACH: R22.1, R23.2, U10.GPIO2/C_ATTACH2/ATTACHMUX2A
- new net DN2_CC1: Q2.D, R7.1, U7.CC1, USB7.CC1
- new net DN2_CC2: Q4.D, R13.1, U7.CC2, USB7.CC2
- new net DN2_D+: R41.2, U10.USB2DN2_D+, USB7.D+
- new net DN2_D-: R44.2, U10.USB2DN2_D-, USB7.D-
- new net DN2_DIR: R19.1, U10.GPIO66/AB2/ATTACHMUX2B, U7.!FLIPPED
- new net DN2_EN/!OC_DET: U10.GPIO19/PRT_CTL2, U7.!OCS, U7.EN, U9.!FAULT
- new net DN2_PWR_EN: R22.2, U7.VBUS_EN/!3.0A, U9.EN
- new net DN2_PWR_EN1: R1.2
- new net DN2_RXA+: U10.USB3DN2_RXA+, USB7.RX1+
- new net DN2_RXA-: U10.USB3DN2_RXA-, USB7.RX1-
- new net DN2_RXB+: U10.USB3DN2_RXB+, USB7.RX2+
- new net DN2_RXB-: U10.USB3DN2_RXB-, USB7.RX2-
- new net DN2_TXA+: U10.USB3DN2_TXA+, USB7.TX1+
- new net DN2_TXA-: U10.USB3DN2_TXA-, USB7.TX1-
- new net DN2_TXB+: U10.USB3DN2_TXB+, USB7.TX2+
- new net DN2_TXB-: U10.USB3DN2_TXB-, USB7.TX2-
- new net DN2_VMON: R26.1, R27.2, U7.VMON
- new net DN3_D+: R36.2, U10.USB2DN3_D+, USB2.D+
- new net DN3_D-: R39.2, U10.USB2DN3_D-, USB2.D-
- new net DN3_EN/!OC_DET: U10.GPIO21/PRT_CTL3, U2.!FAULT, U2.EN
- new net DN3_RX+: U10.USB3DN3_RX+, USB2.RX+
- new net DN3_RX-: U10.USB3DN3_RX-, USB2.RX-
- new net DN3_TX+: U10.USB3DN3_TX+, USB2.TX+
- new net DN3_TX-: U10.USB3DN3_TX-, USB2.TX-
- new net DN4_D+: R42.2, U10.USB2DN4_D+, USB3.D+
- new net DN4_D-: R45.2, U10.USB2DN4_D-, USB3.D-
- new net DN4_EN/!OC_DET: U10.GPIO22/PRT_CTL4, U3.!FAULT, U3.EN
- new net DN4_RX+: U10.USB3DN4_RX+, USB3.RX+
- new net DN4_RX-: U10.USB3DN4_RX-, USB3.RX-
- new net DN4_TX+: U10.USB3DN4_TX+, USB3.TX+
- new net DN4_TX-: U10.USB3DN4_TX-, USB3.TX-
- new net DN5_D+: R37.2, U10.USB2DN5_D+, USB4.D+
- new net DN5_D-: R40.2, U10.USB2DN5_D-, USB4.D-
- new net DN5_EN/!OC_DET: U10.GPIO18/PRT_CTL5, U4.!FAULT, U4.EN
- new net DN6_D+: R43.2, U10.USB2DN6_D+, USB5.D+
- new net DN6_D-: R46.2, U10.USB2DN6_D-, USB5.D-
- new net DN6_EN/!OC_DET: U10.GPIO20/PRT_CTL6/GANG_PWR, U5.!FAULT, U5.EN
- new net GND: C10.C2, C11.C2, C12.C2, C13.C2, C14.C2, C15.C1, C16.C2, C9.C2, R11.1, R2.1, R21.1, R23.1, R25.1, R27.1, R28.1, R3.1, R32.1, R33.1, R34.1, R35.1, R36.1, R37.1, R38.1, R39.1, R40.1, R41.1, R42.1, R43.1, R44.1, R45.1, R46.1, R9.1, U1.!EN_CC, U1.!EN_MUX, U1.GND, U10.GPIO70/ALT_MUX_EN, U10.GPIO71/CC_POL, U10.TESTEN, U10.VSS, U6.VSS@0, U6.VSS@1, U7.VSS@0, U7.VSS@1, USB1.GND, USB1.SHIELD@0, USB1.SHIELD@1, USB1.SHIELD@2, USB1.SHIELD@3, USB2.GND@0, USB2.GND@1, USB2.SHIELD@0, USB2.SHIELD@1, USB3.GND@0, USB3.GND@1, USB3.SHIELD@0, USB3.SHIELD@1, USB4.GND, USB4.SHIELD@0, USB4.SHIELD@1, USB5.GND, USB5.SHIELD@0, USB5.SHIELD@1, USB6.GND, USB6.SHIELD@0, USB6.SHIELD@1, USB6.SHIELD@2, USB6.SHIELD@3, USB7.GND, USB7.SHIELD@0, USB7.SHIELD@1, USB7.SHIELD@2, USB7.SHIELD@3, X1.GND@0, X1.GND@1
- new net I2C_SCL: R30.1, U10.GPIO8/SMBCLK
- new net I2C_SDA: R31.1, U10.GPIO6/SMBDATA
- new net N$1: C1.C2, U1.TX1+
- new net N$10: R3.2, U1.PORT
- new net N$11: C14.C1, U9.VOUT, USB7.VBUS
- new net N$12: C13.C1, R24.2, U8.VOUT, USB6.VBUS
- new net N$13: C9.C1, U2.VOUT, USB2.VBUS
- new net N$14: C12.C1, U5.VOUT, USB5.VBUS
- new net N$15: C11.C1, U4.VOUT, USB4.VBUS
- new net N$16: C10.C1, U3.VOUT, USB3.VBUS
- new net N$17: C16.C1, U10.XTALO, X1.2
- new net N$18: C15.C2, U10.XTALI/CLKIN, X1.1
- new net N$19: R32.2, U10.GPIO12/CFG_STRAP
- new net N$2: C2.C2, U1.TX1-
- new net N$20: R29.1, U10.!RESET
- new net N$21: D2.C, Q2.S, Q4.S
- new net N$22: R28.2, U10.RBIAS
- new net N$23: D1.C, Q1.S, Q3.S
- new net N$24: R10.1, R11.2, U7.CFG_SEL
- new net N$25: R8.1, R9.2, U6.CFG_SEL
- new net N$26: R26.2
- new net N$27: R5.1, U1.DIR
- new net N$3: C3.C2, U1.TX2+
- new net N$4: C4.C2, U1.TX2-
- new net N$5: C5.C2, U1.RX1+
- new net N$6: C6.C2, U1.RX1-
- new net N$7: C7.C2, U1.RX2+
- new net N$8: C8.C2, U1.RX2-
- new net N$9: R4.1, U1.VBUS_DET
- new net SPI_MISO: R33.2, U10.GPIO9/SPI_DI/CFG_BC_EN
- new net SPI_MOSI: U10.GPIO5/SPI_DO
- new net SPI_SCK: U10.GPIO4/SPI_CLK
- new net UP_ATTACH: SJ1.2, U10.GPIO64/C_ATTACH0
- new net UP_CC1: U1.CC1, USB1.CC1
- new net UP_CC2: U1.CC2, USB1.CC2
- new net UP_D+: U10.USB2UP_D+, USB1.D+
- new net UP_D-: U10.USB2UP_D-, USB1.D-
- new net UP_RX+: U1.RX+, U10.USB3UP_RX+
- new net UP_RX-: U1.RX-, U10.USB3UP_RX-
- new net UP_RX1+: C5.C1, USB1.RX1+
- new net UP_RX1-: C6.C1, USB1.RX1-
- new net UP_RX2+: C7.C1, USB1.RX2+
- new net UP_RX2-: C8.C1, USB1.RX2-
- new net UP_TX+: U1.TX+, U10.USB3UP_TX+
- new net UP_TX-: U1.TX-, U10.USB3UP_TX-
- new net UP_TX1+: C1.C1, USB1.TX1+
- new net UP_TX1-: C2.C1, USB1.TX1-
- new net UP_TX2+: C3.C1, USB1.TX2+
- new net UP_TX2-: C4.C1, USB1.TX2-
- new net UP_VBUS_DET: R1.1, R2.2, SJ1.1, U10.GPIO16/VBUS_DET
- new net VBUS: R4.2, USB1.VBUS

Commit message: Work on power
Parts:
- added F1, F2: (no value), PTC Fuses:PTC1812
- added J1: DCJACK, DC Jack:DCJACK
- added R47, R48: 165 Ohms, Resistor:RESISTOR-0603
- added U12: MIC23159, Microchip:MIC23159
- U11: value MIC24045 -> MIC24045-KD; device Microchip:MIC24045 -> Microchip:MIC24045-KD
Connections:
- new net N$28: R47.1, U8.ILIMIT
- new net N$29: R48.1, U9.ILIMIT
- net 5V0: now also F1.1
- net GND: now also R47.2, R48.2, U8.GND, U9.GND
- net VBUS: now also F1.2
Other:
- moved on the sheet: U11
